Commit message: added minor changes to kobuki_description based on icclab/kobuki_ros

File: kobuki_description/urdf/kobuki_gazebo.urdf.xacro (robot description, xacro)
@@ -1,190 +1,197 @@
 <?xml version="1.0"?>
 <robot name="kobuki_sim" xmlns:xacro="http://ros.org/wiki/xacro">
-  <xacro:macro name="kobuki_sim">
-	  <gazebo reference="wheel_left_link">
-	    <mu1>1.0</mu1>
-	    <mu2>1.0</mu2>
-	    <kp>1000000.0</kp>
-	    <kd>100.0</kd>
-	    <minDepth>0.001</minDepth>
-	    <maxVel>1.0</maxVel>
-	  </gazebo>
-	  <gazebo reference="wheel_right_link">
-	    <mu1>1.0</mu1>
-	    <mu2>1.0</mu2>
-	    <kp>1000000.0</kp>
-	    <kd>100.0</kd>
-	    <minDepth>0.001</minDepth>
-	    <maxVel>1.0</maxVel>
-	  </gazebo>
-	  <gazebo reference="caster_front_link">
-	    <mu1>0.0</mu1>
-	    <mu2>0.0</mu2>
-	    <kp>1000000.0</kp>
-	    <kd>100.0</kd>
-	    <minDepth>0.001</minDepth>
-	    <maxVel>1.0</maxVel>
-	  </gazebo>
-	  <gazebo reference="caster_back_link">
-	    <mu1>0.0</mu1>
-	    <mu2>0.0</mu2>
-	    <kp>1000000.0</kp>
-	    <kd>100.0</kd>
-	    <minDepth>0.001</minDepth>
-	    <maxVel>1.0</maxVel>
-	  </gazebo>
-	  <gazebo reference="base_link">
-	    <mu1>0.3</mu1>
-	    <mu2>0.3</mu2>
-	    <sensor type="contact" name="bumpers">
-	      <always_on>1</always_on>
-	      <update_rate>50.0</update_rate>
-	      <visualize>true</visualize>
-	      <contact>
-	        <collision>base_footprint_fixed_joint_lump__base_collision</collision>
-	      </contact>
-	    </sensor>
-	  </gazebo>
-	  <gazebo reference="cliff_sensor_left_link">
-	    <sensor type="ray" name="cliff_sensor_left">
-	      <always_on>true</always_on>
-	      <update_rate>50</update_rate>
-	      <visualize>true</visualize>
-	      <ray>
-	        <scan>
-	          <horizontal>
-	            <samples>50</samples>
-	            <resolution>1.0</resolution>
-	            <min_angle>-0.0436</min_angle>  <!-- -2.5 degree -->
-	            <max_angle>0.0436</max_angle> <!-- 2.5 degree -->
-	          </horizontal>
-			<!-- Can't use vertical rays until this bug is resolved -->
-			<!-- https://bitbucket.org/osrf/gazebo/issue/509/vertical-sensor-doesnt-works -->
-			<!-- <vertical> -->
-			<!--     <samples>50</samples> -->
-			<!--     <resolution>1.0</resolution> -->
-			<!--     <min_angle>-0.0436</min_angle>  -2.5 degree -->
-			<!--     <max_angle>0.0436</max_angle> 2.5 degree -->
-			<!-- </vertical> -->
-	        </scan>
-	        <range>
-	          <min>0.01</min>
-	          <max>0.15</max>
-	          <resolution>1.0</resolution>
-	        </range>
-	      </ray>
-	    </sensor>
-	  </gazebo>
-	  <gazebo reference="cliff_sensor_right_link">
-	    <sensor type="ray" name="cliff_sensor_right">
-	      <always_on>true</always_on>
-	      <update_rate>50</update_rate>
-	      <visualize>true</visualize>
-	      <ray>
-	        <scan>
-	          <horizontal>
-	            <samples>50</samples>
-	            <resolution>1.0</resolution>
-	            <min_angle>-0.0436</min_angle>  <!-- -2.5 degree -->
-	            <max_angle>0.0436</max_angle> <!-- 2.5 degree -->
-	          </horizontal>
-			<!-- Can't use vertical rays until this bug is resolved -->
-			<!-- https://bitbucket.org/osrf/gazebo/issue/509/vertical-sensor-doesnt-works -->
-			<!-- <vertical> -->
-			<!--     <samples>50</samples> -->
-			<!--     <resolution>1.0</resolution> -->
-			<!--     <min_angle>-0.0436</min_angle>  -2.5 degree -->
-			<!--     <max_angle>0.0436</max_angle> 2.5 degree -->
-			<!-- </vertical> -->
-	        </scan>
-	        <range>
-	          <min>0.01</min>
-	          <max>0.15</max>
-	          <resolution>1.0</resolution>
-	        </range>
-	      </ray>
-	    </sensor>
-	  </gazebo>
-	  <gazebo reference="cliff_sensor_front_link">
-	    <sensor type="ray" name="cliff_sensor_front">
-	      <always_on>true</always_on>
-	      <update_rate>50</update_rate>
-	      <visualize>true</visualize>
-	      <ray>
-	        <scan>
-	          <horizontal>
-	            <samples>50</samples>
-	            <resolution>1.0</resolution>
-	            <min_angle>-0.0436</min_angle>  <!-- -2.5 degree -->
-	            <max_angle>0.0436</max_angle> <!-- 2.5 degree -->
-	          </horizontal>
-			<!-- Can't use vertical rays until this bug is resolved -->
-			<!-- https://bitbucket.org/osrf/gazebo/issue/509/vertical-sensor-doesnt-works -->
-			<!-- <vertical> -->
-			<!--     <samples>50</samples> -->
-			<!--     <resolution>1.0</resolution> -->
-			<!--     <min_angle>-0.0436</min_angle>  -2.5 degree -->
-			<!--     <max_angle>0.0436</max_angle> 2.5 degree -->
-			<!-- </vertical> -->
-	        </scan>
-	        <range>
-	          <min>0.01</min>
-	          <max>0.15</max>
-	          <resolution>1.0</resolution>
-	        </range>
-	      </ray>
-	    </sensor>
-	  </gazebo>
-	  <gazebo reference="gyro_link">
-	   <sensor type="imu" name="imu">
-        <plugin name="gazebo_ros_imu_controller" filename="libgazebo_ros_imu_sensor.so">
-          <ros>
-            <argument>~/out:=imu</argument>
-          </ros>
-          <output_type>sensor_msgs/msg/Imu</output_type>
-          <body_name>gyro_link</body_name>
-          <frame_name>gyro_link</frame_name>
-        </plugin>
-        <always_on>true</always_on>
-        <update_rate>50</update_rate>
-        <visualize>false</visualize>
-        <imu>
-          <noise>
-            <type>gaussian</type>
-	          <rate>
-	            <mean>0.0</mean>
-	            <stddev>${0.0014*0.0014}</stddev> <!-- 0.25 x 0.25 (deg/s) -->
-	            <bias_mean>0.0</bias_mean>
-	            <bias_stddev>0.0</bias_stddev>
-	          </rate>
-		        <accel> <!-- not used in the plugin and real robot, hence using tutorial values -->
-			        <mean>0.0</mean>
-			        <stddev>1.7e-2</stddev>
-			        <bias_mean>0.1</bias_mean>
-			        <bias_stddev>0.001</bias_stddev>
-		        </accel>
-          </noise>
-	      </imu>
-      </sensor>
-	  </gazebo>
-	  <gazebo>
-      <plugin name="differential_drive_controller" filename="libgazebo_ros_diff_drive.so">
-        <update_rate>30</update_rate>
-        <left_joint>wheel_left_joint</left_joint>
-        <right_joint>wheel_right_joint</right_joint>
-        <wheel_separation>0.230</wheel_separation>
-        <wheel_diameter>0.070</wheel_diameter>
-        <max_wheel_torque>1.0</max_wheel_torque>
-        <max_wheel_acceleration>1.0</max_wheel_acceleration>
-        <command_topic>cmd_vel</command_topic>
-        <!-- output -->
-        <publish_odom>true</publish_odom>
-        <publish_odom_tf>true</publish_odom_tf>
-        <publish_wheel_tf>true</publish_wheel_tf>
-        <odometry_topic>odom</odometry_topic>
-        <odometry_frame>odom</odometry_frame>
-        <robot_base_frame>base_footprint</robot_base_frame>
-	    </plugin>
-	  </gazebo>
-  </xacro:macro>
+	<xacro:arg name="namespace" default=""/>
+	<xacro:property name="robot_namespace" value="/$(arg namespace)"/>
+	<xacro:macro name="kobuki_sim">
+		<gazebo reference="wheel_left_link">
+			<mu1>1.0</mu1>
+			<mu2>1.0</mu2>
+			<kp>1000000.0</kp>
+			<kd>100.0</kd>
+			<minDepth>0.001</minDepth>
+			<maxVel>1.0</maxVel>
+		</gazebo>
+		<gazebo reference="wheel_right_link">
+			<mu1>1.0</mu1>
+			<mu2>1.0</mu2>
+			<kp>1000000.0</kp>
+			<kd>100.0</kd>
+			<minDepth>0.001</minDepth>
+			<maxVel>1.0</maxVel>
+		</gazebo>
+		<gazebo reference="caster_front_link">
+			<mu1>0.0</mu1>
+			<mu2>0.0</mu2>
+			<kp>1000000.0</kp>
+			<kd>100.0</kd>
+			<minDepth>0.001</minDepth>
+			<maxVel>1.0</maxVel>
+		</gazebo>
+		<gazebo reference="caster_back_link">
+			<mu1>0.0</mu1>
+			<mu2>0.0</mu2>
+			<kp>1000000.0</kp>
+			<kd>100.0</kd>
+			<minDepth>0.001</minDepth>
+			<maxVel>1.0</maxVel>
+		</gazebo>
+		<gazebo reference="base_link">
+			<mu1>0.3</mu1>
+			<mu2>0.3</mu2>
+			<sensor type="contact" name="bumpers">
+			<always_on>1</always_on>
+			<update_rate>50.0</update_rate>
+			<visualize>true</visualize>
+			<contact>
+				<collision>base_footprint_fixed_joint_lump__base_collision</collision>
+			</contact>
+			</sensor>
+		</gazebo>
+		<gazebo reference="cliff_sensor_left_link">
+			<sensor type="ray" name="cliff_sensor_left">
+			<always_on>true</always_on>
+			<update_rate>50</update_rate>
+			<visualize>true</visualize>
+			<ray>
+				<scan>
+				<horizontal>
+					<samples>50</samples>
+					<resolution>1.0</resolution>
+					<min_angle>-0.0436</min_angle>  <!-- -2.5 degree -->
+					<max_angle>0.0436</max_angle> <!-- 2.5 degree -->
+				</horizontal>
+				<!-- Can't use vertical rays until this bug is resolved -->
+				<!-- https://bitbucket.org/osrf/gazebo/issue/509/vertical-sensor-doesnt-works -->
+				<!-- <vertical> -->
+				<!--     <samples>50</samples> -->
+				<!--     <resolution>1.0</resolution> -->
+				<!--     <min_angle>-0.0436</min_angle>  -2.5 degree -->
+				<!--     <max_angle>0.0436</max_angle> 2.5 degree -->
+				<!-- </vertical> -->
+				</scan>
+				<range>
+				<min>0.01</min>
+				<max>0.15</max>
+				<resolution>1.0</resolution>
+				</range>
+			</ray>
+			</sensor>
+		</gazebo>
+		<gazebo reference="cliff_sensor_right_link">
+			<sensor type="ray" name="cliff_sensor_right">
+			<always_on>true</always_on>
+			<update_rate>50</update_rate>
+			<visualize>true</visualize>
+			<ray>
+				<scan>
+				<horizontal>
+					<samples>50</samples>
+					<resolution>1.0</resolution>
+					<min_angle>-0.0436</min_angle>  <!-- -2.5 degree -->
+					<max_angle>0.0436</max_angle> <!-- 2.5 degree -->
+				</horizontal>
+				<!-- Can't use vertical rays until this bug is resolved -->
+				<!-- https://bitbucket.org/osrf/gazebo/issue/509/vertical-sensor-doesnt-works -->
+				<!-- <vertical> -->
+				<!--     <samples>50</samples> -->
+				<!--     <resolution>1.0</resolution> -->
+				<!--     <min_angle>-0.0436</min_angle>  -2.5 degree -->
+				<!--     <max_angle>0.0436</max_angle> 2.5 degree -->
+				<!-- </vertical> -->
+				</scan>
+				<range>
+				<min>0.01</min>
+				<max>0.15</max>
+				<resolution>1.0</resolution>
+				</range>
+			</ray>
+			</sensor>
+		</gazebo>
+		<gazebo reference="cliff_sensor_front_link">
+			<sensor type="ray" name="cliff_sensor_front">
+			<always_on>true</always_on>
+			<update_rate>50</update_rate>
+			<visualize>true</visualize>
+			<ray>
+				<scan>
+				<horizontal>
+					<samples>50</samples>
+					<resolution>1.0</resolution>
+					<min_angle>-0.0436</min_angle>  <!-- -2.5 degree -->
+					<max_angle>0.0436</max_angle> <!-- 2.5 degree -->
+				</horizontal>
+				<!-- Can't use vertical rays until this bug is resolved -->
+				<!-- https://bitbucket.org/osrf/gazebo/issue/509/vertical-sensor-doesnt-works -->
+				<!-- <vertical> -->
+				<!--     <samples>50</samples> -->
+				<!--     <resolution>1.0</resolution> -->
+				<!--     <min_angle>-0.0436</min_angle>  -2.5 degree -->
+				<!--     <max_angle>0.0436</max_angle> 2.5 degree -->
+				<!-- </vertical> -->
+				</scan>
+				<range>
+				<min>0.01</min>
+				<max>0.15</max>
+				<resolution>1.0</resolution>
+				</range>
+			</ray>
+			</sensor>
+		</gazebo>
+		<gazebo reference="gyro_link">
+		<sensor type="imu" name="imu">
+			<plugin name="gazebo_ros_imu_controller" filename="libgazebo_ros_imu_sensor.so">
+			<ros>
+				<argument>~/out:=imu</argument>
+			</ros>
+			<output_type>sensor_msgs/msg/Imu</output_type>
+			<body_name>gyro_link</body_name>
+			<frame_name>gyro_link</frame_name>
+			</plugin>
+			<always_on>true</always_on>
+			<update_rate>50</update_rate>
+			<visualize>false</visualize>
+			<imu>
+			<noise>
+				<type>gaussian</type>
+				<rate>
+					<mean>0.0</mean>
+					<stddev>${0.0014*0.0014}</stddev> <!-- 0.25 x 0.25 (deg/s) -->
+					<bias_mean>0.0</bias_mean>
+					<bias_stddev>0.0</bias_stddev>
+				</rate>
+					<accel> <!-- not used in the plugin and real robot, hence using tutorial values -->
+						<mean>0.0</mean>
+						<stddev>1.7e-2</stddev>
+						<bias_mean>0.1</bias_mean>
+						<bias_stddev>0.001</bias_stddev>
+					</accel>
+			</noise>
+			</imu>
+		</sensor>
+		</gazebo>
+		<gazebo>
+			<plugin name="differential_drive_controller" filename="libgazebo_ros_diff_drive.so">
+				<update_rate>30</update_rate>
+				<ros>
+					<namespace>${robot_namespace}</namespace>
+					<remapping>/tf:=tf</remapping>
+					<remapping>/tf_static:=tf_static</remapping>
+				</ros>
+				<left_joint>wheel_left_joint</left_joint>
+				<right_joint>wheel_right_joint</right_joint>
+				<wheel_separation>0.230</wheel_separation>
+				<wheel_diameter>0.070</wheel_diameter>
+				<max_wheel_torque>1.0</max_wheel_torque>
+				<max_wheel_acceleration>1.0</max_wheel_acceleration>
+				<command_topic>cmd_vel</command_topic>
+				<!-- output -->
+				<publish_odom>true</publish_odom>
+				<publish_odom_tf>true</publish_odom_tf>
+				<publish_wheel_tf>true</publish_wheel_tf>
+				<odometry_topic>odom</odometry_topic>
+				<odometry_frame>odom</odometry_frame>
+				<robot_base_frame>base_footprint</robot_base_frame>
+			</plugin>
+		</gazebo>
+	</xacro:macro>
 </robot>
