Commit message: changed kobuki_gaebo

File: kobuki_description/urdf/kobuki.urdf.xacro (robot description, xacro)
@@ -23,6 +23,6 @@
     <joint name="base_joint" type="fixed">
       <origin xyz="0 0 0.0102" rpy="0 0 0" />
-      <parent link="base_footprint"/>
-      <child link="base_link" />
+      <parent link="base_link"/>
+      <child link="base_footprint" />
     </joint>
     <link name="base_link">

File: kobuki_description/urdf/kobuki_gazebo.urdf.xacro (robot description, xacro)
@@ -223,4 +223,5 @@
 					<remapping>/tf:=tf</remapping>
 					<remapping>/tf_static:=tf_static</remapping>
+					<remapping>/cmd_vel:=commands/velocity</remapping>
 				</ros>
 				<left_joint>wheel_left_joint</left_joint>

Commit message: added modifications from michieletto/kobuki_ros

File: kobuki_description/urdf/kobuki.urdf.xacro (robot description, xacro)
@@ -208,4 +208,10 @@
       </inertial>
     </link>
+    <joint name="camera_joint" type="fixed">
+      <origin xyz="0.037 -0.002 0.559" rpy="0.0003 0.5032 -0.0309" />
+      <parent link="base_footprint"/>
+      <child link="camera_link" />
+    </joint>
+    <link name="camera_link"/>
     <!-- Kobuki Gazebo simulation details -->
     <xacro:kobuki_sim/>
